File: PCB's/KiCad Project Files/Front PCB/Game Controller - Front PCB.kicad_sch (KiCad schematic)
At the start: 54 parts, among them M1_N1 MOSI, M1_P1 MOSI, M2_N1 MOSI, M2_P1 MOSI, Q1 2N7002, Q2 2N7002, SW1 A, SW2 B, SW3 X, SW4 Y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

Commit message: Updated front PCB drawing and kicad project files
Connections:
- net VCC: now also D1.1 (BA); no longer D1.4 (K)
- net at U7.3 (OUTB): now also D1.4 (K); no longer D1.1 (BA)
Other:
- note added: "Note: Pads 4+1 Swapped to allow mounting on rear face of PCB"
Changed lines of the file:
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@@
 	(wire
 		(pts
-			(xy 294.64 233.68) (xy 300.99 233.68)
+			(xy 317.5 233.68) (xy 317.5 231.14)
+		)
+		(stroke
+			(width 0)
+			(type default)
+		)
+	)
+	(wire
+		(pts
+			(xy 294.64 233.68) (xy 317.5 233.68)
 		)
 		(stroke
@@
 	(wire
 		(pts
+			(xy 303.53 247.65) (xy 298.45 247.65)
+		)
+		(stroke
+			(width 0)
+			(type default)
+		)
+	)
+	(wire
+		(pts
 			(xy 300.99 226.06) (xy 300.99 228.6)
 		)
@@
 	(wire
 		(pts
-			(xy 317.5 228.6) (xy 317.5 231.14)
-		)
-		(stroke
-			(width 0)
-			(type default)
-		)
-	)
-	(wire
-		(pts
 			(xy 124.46 259.08) (xy 120.65 259.08)
 		)
@@
 	(wire
 		(pts
-			(xy 300.99 233.68) (xy 300.99 236.22)
-		)
-		(stroke
-			(width 0)
-			(type default)
-		)
-	)
-	(wire
-		(pts
 			(xy 247.65 110.49) (xy 247.65 121.92)
 		)
@@
 	(wire
 		(pts
-			(xy 300.99 236.22) (xy 303.53 236.22)
-		)
-		(stroke
-			(width 0)
-			(type default)
-		)
-	)
-	(wire
-		(pts
 			(xy 115.57 201.93) (xy 118.11 201.93)
 		)
@@
 	(wire
 		(pts
+			(xy 298.45 247.65) (xy 298.45 245.11)
+		)
+		(stroke
+			(width 0)
+			(type default)
+		)
+	)
+	(wire
+		(pts
 			(xy 252.73 228.6) (xy 259.08 228.6)
 		)
@@
 	(wire
 		(pts
+			(xy 303.53 236.22) (xy 303.53 247.65)
+		)
+		(stroke
+			(width 0)
+			(type default)
+		)
+	)
+	(wire
+		(pts
 			(xy 335.28 71.12) (xy 335.28 73.66)
 		)
@@
 		)
 	)
+	(text "Note: Pads 4+1 Swapped to \nallow mounting on rear \nface of PCB"
+		(exclude_from_sim no)
+		(at 321.31 243.586 0)
+		(effects
+			(font
+				(size 1.27 1.27)
+			)
+		)
+	)
 	(label "DOWN"
 		(at 118.11 219.71 0)
@@
 	)
 	(symbol
+		(lib_id "power:VCC")
+		(at 298.45 245.11 0)
+		(unit 1)
+		(exclude_from_sim no)
+		(in_bom yes)
+		(on_board yes)
+		(dnp no)
+		(fields_autoplaced yes)
+		(property "Reference" "#PWR020"
+			(at 298.45 248.92 0)
+			(effects
+				(font
+					(size 1.27 1.27)
+				)
+				(hide yes)
+			)
+		)
+		(property "Value" "VCC"
+			(at 298.45 240.03 0)
+			(effects
+				(font
+					(size 1.27 1.27)
+				)
+			)
+		)
+		(property "Footprint" ""
+			(at 298.45 245.11 0)
+			(effects
+				(font
+					(size 1.27 1.27)
+				)
+				(hide yes)
+			)
+		)
+		(property "Datasheet" ""
+			(at 298.45 245.11 0)
+			(effects
+				(font
+					(size 1.27 1.27)
+				)
+				(hide yes)
+			)
+		)
+		(property "Description" ""
+			(at 298.45 245.11 0)
+			(effects
+				(font
+					(size 1.27 1.27)
+				)
+				(hide yes)
+			)
+		)
+		(pin "1"
+		)
+		(instances
+			(project "Game Controller - Front PCB"
+				(path "/ff343239-2598-48f4-ac52-06d80fe426a2"
+					(reference "#PWR020")
+					(unit 1)
+				)
+			)
+		)
+	)
+	(symbol
 		(lib_id "Device:C")
 		(at 60.96 167.64 90)
@@
 					(unit 1)
 				)
-			)
-		)
-	)
-	(symbol
-		(lib_id "power:VCC")
-		(at 317.5 228.6 0)
-		(unit 1)
-		(exclude_from_sim no)
-		(in_bom yes)
-		(on_board yes)
-		(dnp no)
-		(fields_autoplaced yes)
-		(property "Reference" "#PWR023"
-			(at 317.5 232.41 0)
-			(effects
-				(font
-					(size 1.27 1.27)
-				)
-				(hide yes)
-			)
-		)
-		(property "Value" "VCC"
-			(at 317.5 223.52 0)
-			(effects
-				(font
-					(size 1.27 1.27)
-				)
-			)
-		)
-		(property "Footprint" ""
-			(at 317.5 228.6 0)
-			(effects
-				(font
-					(size 1.27 1.27)
-				)
-				(hide yes)
-			)
-		)
-		(property "Datasheet" ""
-			(at 317.5 228.6 0)
-			(effects
-				(font
-					(size 1.27 1.27)
-				)
-				(hide yes)
-			)
-		)
-		(property "Description" ""
-			(at 317.5 228.6 0)
-			(effects
-				(font
-					(size 1.27 1.27)
-				)
-				(hide yes)
-			)
-		)
-		(pin "1"
-		)
-		(instances
-			(project "Game Controller - Front PCB"
-				(path "/ff343239-2598-48f4-ac52-06d80fe426a2"
-					(reference "#PWR023")
-					(unit 1)
-				)
